File: Hardware/OpenBook_PCB.brd (EAGLE design)
At the start: 170.2 x 111.3 mm, 103 parts, among them IC1 BD5229G-TR, IC4 XC6220A331MR-G, J1 FH34SRJ-24S-0.5SH_99_, J2 SAMACSYS_PARTS_USB4110-GF-A, J3 QWIIC_RIGHT_ANGLE, J4 112A-TAAR-R03_ATTEND, Q1 20V/4.2A/52mΩ/1.4W, Q2 20V/4.2A/52mΩ/1.4W, Q3 SI1308EDL-T1-GE3, U1 W25Q512JVEIQ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

Commit message: Add files via upload
Parts:
- moved TP11 15.8 mm to (11.2, 3.81)
- moved TP9 8.10 mm to (7.11, 7.37)
Routing:
- net SRC: track 38.7 -> 67.0 mm, vias 2 -> 0
- net N$8: track 43.3 -> 18.8 mm, vias 2 -> 4
- net USB_D+: track 166.3 -> 142.2 mm, vias 2 -> 4
- net RESE': track 19.8 -> 1.85 mm, vias 2 -> 0
- net EPD_BUSY: track 126.0 -> 136.1 mm, vias 6 -> 4
- net EPD_RST: track 107.4 -> 117.1 mm, vias 6 -> 4
- net MOSI: track 159.4 -> 150.1 mm, vias 5 -> 6
- net MISO: track 113.9 -> 106.1 mm
- net EPD_CS: track 94.4 -> 100.1 mm, vias 5 -> 4
- net SCK: track 162.4 -> 159.1 mm, vias 6 -> 7
- net 32KHZ: track 87.1 -> 89.9 mm, vias 3 -> 4
- net EPD_DC: track 112.3 -> 115.1 mm
- net RESE: track 26.7 -> 25.0 mm, vias 3 -> 2
- net SCL: track 212.9 -> 211.4 mm
- net GDR: track 28.4 -> 29.7 mm
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